File: serprog.sch (KiCad schematic (older format))
At the start: 44 parts, among them J1 USB_B_Micro, J2 Conn_01x04, SW1 SW_Push_SPDT, U1 TXS0108EPW, U2 XC6206PxxxMR1v8, U3 XC6206PxxxMR3v3, U4 AT25xxx, U5 STM32F102R8Tx, Y1 8M

Commit message: v0.1
Parts:
- removed J2: Conn_01x04, Connector_PinHeader_2.54mm:PinHeader_1x04_P2.54mm_Vertical, symbol Connector_Generic:Conn_01x04
- J1: footprint Connector_USB:USB_Micro-B_Molex_47346-0001 -> Connector_USB:USB_Micro-B_Molex-105017-0001
Connections:
- net +3V3: now also TP2.1
- net FLASH_MISO: no longer TP3.1
- net FLASH_MOSI: no longer TP4.1
- net FLASH_NSS: no longer TP1.1
- net FLASH_SCK: no longer TP2.1
- net GND: now also TP1.1
- net USART1_RX: now also TP4.1
- net USART1_TX: now also TP3.1
Changed lines of the file:
@@
 F 0 "J1" H 3107 1717 50  0000 C CNN
 F 1 "USB_B_Micro" H 3107 1626 50  0000 C CNN
-F 2 "Connector_USB:USB_Micro-B_Molex_47346-0001" H 3200 1200 50  0001 C CNN
+F 2 "Connector_USB:USB_Micro-B_Molex-105017-0001" H 3200 1200 50  0001 C CNN
 F 3 "~" H 3200 1200 50  0001 C CNN
 	1    3050 1250
@@
 	5700 5600 5650 5600
 $Comp
-L Connector_Generic:Conn_01x04 J2
-U 1 1 60B0554E
-P 5450 5500
-F 0 "J2" H 5530 5492 50  0000 L CNN
-F 1 "Conn_01x04" H 5530 5401 50  0000 L CNN
-F 2 "Connector_PinHeader_2.54mm:PinHeader_1x04_P2.54mm_Vertical" H 5450 5500 50  0001 C CNN
-F 3 "~" H 5450 5500 50  0001 C CNN
-	1    5450 5500
-	-1   0    0    1
-$EndComp
-$Comp
 L Memory_EEPROM:AT25xxx U4
 U 1 1 60968DAB
@@
 NoConn ~ 8900 4800
 $Comp
-L Connector:TestPoint TP1
-U 1 1 6104E09E
-P 4200 3550
-F 0 "TP1" V 4150 3700 50  0000 L CNN
-F 1 "TestPoint" V 4245 3738 50  0001 L CNN
-F 2 "TestPoint:TestPoint_Pad_D1.0mm" H 4400 3550 50  0001 C CNN
-F 3 "~" H 4400 3550 50  0001 C CNN
-	1    4200 3550
-	0    1    1    0
-$EndComp
-$Comp
-L Connector:TestPoint TP2
-U 1 1 61054E74
-P 4200 3650
-F 0 "TP2" V 4150 3800 50  0000 L CNN
-F 1 "TestPoint" V 4245 3838 50  0001 L CNN
-F 2 "TestPoint:TestPoint_Pad_D1.0mm" H 4400 3650 50  0001 C CNN
-F 3 "~" H 4400 3650 50  0001 C CNN
-	1    4200 3650
-	0    1    1    0
-$EndComp
-$Comp
-L Connector:TestPoint TP3
-U 1 1 610553C8
-P 4200 3750
-F 0 "TP3" V 4150 3900 50  0000 L CNN
-F 1 "TestPoint" V 4245 3938 50  0001 L CNN
-F 2 "TestPoint:TestPoint_Pad_D1.0mm" H 4400 3750 50  0001 C CNN
-F 3 "~" H 4400 3750 50  0001 C CNN
-	1    4200 3750
-	0    1    1    0
-$EndComp
-$Comp
-L Connector:TestPoint TP4
-U 1 1 6105576F
-P 4200 3850
-F 0 "TP4" V 4150 4000 50  0000 L CNN
-F 1 "TestPoint" V 4245 4038 50  0001 L CNN
-F 2 "TestPoint:TestPoint_Pad_D1.0mm" H 4400 3850 50  0001 C CNN
-F 3 "~" H 4400 3850 50  0001 C CNN
-	1    4200 3850
-	0    1    1    0
-$EndComp
-Wire Wire Line
-	3850 3550 4200 3550
-Wire Wire Line
-	3950 3650 4200 3650
-Wire Wire Line
-	4050 3750 4200 3750
-Wire Wire Line
-	4150 3850 4200 3850
-$Comp
 L Device:R R1
 U 1 1 6107DD48
@@
 Text GLabel 4100 2750 0    50   Input ~ 0
 FLASH_VCC
+$Comp
+L Connector:TestPoint TP1
+U 1 1 6092BE60
+P 5650 5300
+F 0 "TP1" V 5650 5550 50  0000 C CNN
+F 1 "TestPoint" V 5754 5372 50  0001 C CNN
+F 2 "TestPoint:TestPoint_Pad_D1.0mm" H 5850 5300 50  0001 C CNN
+F 3 "~" H 5850 5300 50  0001 C CNN
+	1    5650 5300
+	0    -1   -1   0
+$EndComp
+$Comp
+L Connector:TestPoint TP2
+U 1 1 609307F4
+P 5650 5400
+F 0 "TP2" V 5650 5650 50  0000 C CNN
+F 1 "TestPoint" V 5754 5472 50  0001 C CNN
+F 2 "TestPoint:TestPoint_Pad_D1.0mm" H 5850 5400 50  0001 C CNN
+F 3 "~" H 5850 5400 50  0001 C CNN
+	1    5650 5400
+	0    -1   -1   0
+$EndComp
+$Comp
+L Connector:TestPoint TP3
+U 1 1 60930D0E
+P 5650 5500
+F 0 "TP3" V 5650 5750 50  0000 C CNN
+F 1 "TestPoint" V 5754 5572 50  0001 C CNN
+F 2 "TestPoint:TestPoint_Pad_D1.0mm" H 5850 5500 50  0001 C CNN
+F 3 "~" H 5850 5500 50  0001 C CNN
+	1    5650 5500
+	0    -1   -1   0
+$EndComp
+$Comp
+L Connector:TestPoint TP4
+U 1 1 60931275
+P 5650 5600
+F 0 "TP4" V 5650 5850 50  0000 C CNN
+F 1 "TestPoint" V 5754 5672 50  0001 C CNN
+F 2 "TestPoint:TestPoint_Pad_D1.0mm" H 5850 5600 50  0001 C CNN
+F 3 "~" H 5850 5600 50  0001 C CNN
+	1    5650 5600
+	0    -1   -1   0
+$EndComp
 $EndSCHEMATC

Commit message: delete useless testpad
Parts:
- removed TP2: TestPoint, TestPoint:TestPoint_Pad_D1.0mm, symbol Connector:TestPoint
- TP1: value TestPoint -> GND
- TP2: renamed from TP3; value TestPoint -> TX
- TP3: renamed from TP4; value TestPoint -> RX
Other:
- moved on the sheet: TP1
Changed lines of the file:
@@
 NoConn ~ 8900 3400
 Wire Wire Line
-	5700 5300 5650 5300
+	5700 5400 5650 5400
 $Comp
 L power:GND #PWR017
 U 1 1 60B1D5EA
-P 5700 5300
-F 0 "#PWR017" H 5700 5050 50  0001 C CNN
-F 1 "GND" V 5705 5172 50  0000 R CNN
-F 2 "" H 5700 5300 50  0001 C CNN
-F 3 "" H 5700 5300 50  0001 C CNN
-	1    5700 5300
-	0    -1   -1   0
-$EndComp
-Wire Wire Line
-	5700 5400 5650 5400
-$Comp
-L power:+3.3V #PWR018
-U 1 1 60B14F4D
 P 5700 5400
-F 0 "#PWR018" H 5700 5250 50  0001 C CNN
-F 1 "+3.3V" V 5715 5528 50  0000 L CNN
+F 0 "#PWR017" H 5700 5150 50  0001 C CNN
+F 1 "GND" V 5705 5272 50  0000 R CNN
 F 2 "" H 5700 5400 50  0001 C CNN
 F 3 "" H 5700 5400 50  0001 C CNN
 	1    5700 5400
-	0    1    1    0
+	0    -1   -1   0
 $EndComp
 Wire Wire Line
@@
 L Connector:TestPoint TP1
 U 1 1 6092BE60
-P 5650 5300
-F 0 "TP1" V 5650 5550 50  0000 C CNN
-F 1 "TestPoint" V 5754 5372 50  0001 C CNN
-F 2 "TestPoint:TestPoint_Pad_D1.0mm" H 5850 5300 50  0001 C CNN
-F 3 "~" H 5850 5300 50  0001 C CNN
-	1    5650 5300
-	0    -1   -1   0
-$EndComp
-$Comp
-L Connector:TestPoint TP2
-U 1 1 609307F4
 P 5650 5400
-F 0 "TP2" V 5650 5650 50  0000 C CNN
-F 1 "TestPoint" V 5754 5472 50  0001 C CNN
+F 0 "TP1" V 5650 5650 50  0000 C CNN
+F 1 "GND" V 5754 5472 50  0001 C CNN
 F 2 "TestPoint:TestPoint_Pad_D1.0mm" H 5850 5400 50  0001 C CNN
 F 3 "~" H 5850 5400 50  0001 C CNN
@@
 $EndComp
 $Comp
-L Connector:TestPoint TP3
+L Connector:TestPoint TP2
 U 1 1 60930D0E
 P 5650 5500
-F 0 "TP3" V 5650 5750 50  0000 C CNN
-F 1 "TestPoint" V 5754 5572 50  0001 C CNN
+F 0 "TP2" V 5650 5750 50  0000 C CNN
+F 1 "TX" V 5754 5572 50  0001 C CNN
 F 2 "TestPoint:TestPoint_Pad_D1.0mm" H 5850 5500 50  0001 C CNN
 F 3 "~" H 5850 5500 50  0001 C CNN
@@
 $EndComp
 $Comp
-L Connector:TestPoint TP4
+L Connector:TestPoint TP3
 U 1 1 60931275
 P 5650 5600
-F 0 "TP4" V 5650 5850 50  0000 C CNN
-F 1 "TestPoint" V 5754 5672 50  0001 C CNN
+F 0 "TP3" V 5650 5850 50  0000 C CNN
+F 1 "RX" V 5754 5672 50  0001 C CNN
 F 2 "TestPoint:TestPoint_Pad_D1.0mm" H 5850 5600 50  0001 C CNN
 F 3 "~" H 5850 5600 50  0001 C CNN

Commit message: v0.2
Parts:
- removed U1: TXS0108EPW, Package_SO:TSSOP-20_4.4x6.5mm_P0.65mm, symbol Logic_LevelTranslator:TXS0108EPW
- added U1: TXB0104PW, Package_SO:TSSOP-14_4.4x5mm_P0.65mm, symbol Logic_LevelTranslator:TXB0104PW
Connections:
- net +3V3: now also U1.14 (VCCB)
- net FLASH_MISO: now also U1.4 (A3)
- net FLASH_MOSI: now also U1.5 (A4)
- net FLASH_NSS: now also U1.2 (A1)
- net FLASH_SCK: now also U1.3 (A2)
- net FLASH_VCC: now also U1.1 (VCCA)
- net GND: now also U1.7 (GND)
- net SPI1_MISO: now also U1.11 (B3)
- net SPI1_MOSI: now also U1.10 (B4)
- net SPI1_NSS: now also U1.13 (B1)
- net SPI1_SCK: now also U1.12 (B2)
- net at R8.2: now also U1.8 (OE)
- no-connect marks 47 -> 39
Changed lines of the file:
@@
 	3600 5250 3700 5250
 $Comp
-L power:+3.3V #PWR026
+L power:+3.3V #PWR025
 U 1 1 60A418C5
 P 8000 1300
-F 0 "#PWR026" H 8000 1150 50  0001 C CNN
+F 0 "#PWR025" H 8000 1150 50  0001 C CNN
 F 1 "+3.3V" H 8015 1473 50  0000 C CNN
 F 2 "" H 8000 1300 50  0001 C CNN
@@
 	8100 1400 8200 1400
 $Comp
-L power:GND #PWR027
+L power:GND #PWR026
 U 1 1 60A4D3BD
 P 8000 5300
-F 0 "#PWR027" H 8000 5050 50  0001 C CNN
+F 0 "#PWR026" H 8000 5050 50  0001 C CNN
 F 1 "GND" H 8005 5127 50  0000 C CNN
 F 2 "" H 8000 5300 50  0001 C CNN
@@
 	6100 6500 6400 6500
 $Comp
-L power:+3.3V #PWR024
+L power:+3.3V #PWR023
 U 1 1 60A95BE4
 P 6400 5950
-F 0 "#PWR024" H 6400 5800 50  0001 C CNN
+F 0 "#PWR023" H 6400 5800 50  0001 C CNN
 F 1 "+3.3V" H 6400 6100 50  0000 C CNN
 F 2 "" H 6400 5950 50  0001 C CNN
@@
 $EndComp
 $Comp
-L power:GND #PWR025
+L power:GND #PWR024
 U 1 1 60A96AE9
 P 6400 6500
-F 0 "#PWR025" H 6400 6250 50  0001 C CNN
+F 0 "#PWR024" H 6400 6250 50  0001 C CNN
 F 1 "GND" H 6405 6327 50  0000 C CNN
 F 2 "" H 6400 6500 50  0001 C CNN
@@
 Text GLabel 2750 3550 0    50   Input ~ 0
 SPI1_NSS
-Text GLabel 2750 3650 0    50   Input ~ 0
+Text GLabel 2750 3750 0    50   Input ~ 0
 SPI1_SCK
-Text GLabel 2750 3750 0    50   Input ~ 0
+Text GLabel 2750 3950 0    50   Input ~ 0
 SPI1_MISO
-Text GLabel 2750 3850 0    50   Input ~ 0
+Text GLabel 2750 4150 0    50   Input ~ 0
 SPI1_MOSI
 $Comp
@@
 	5300 4350 5300 4150
 $Comp
-L power:+3.3V #PWR021
+L power:+3.3V #PWR020
 U 1 1 60A68DEC
 P 6000 3700
-F 0 "#PWR021" H 6000 3550 50  0001 C CNN
+F 0 "#PWR020" H 6000 3550 50  0001 C CNN
 F 1 "+3.3V" V 6000 3950 50  0000 C CNN
 F 2 "" H 6000 3700 50  0001 C CNN
@@
 $EndComp
 $Comp
-L power:+1V8 #PWR022
+L power:+1V8 #PWR021
 U 1 1 60A6EB3A
 P 6000 3900
-F 0 "#PWR022" H 6000 3750 50  0001 C CNN
+F 0 "#PWR021" H 6000 3750 50  0001 C CNN
 F 1 "+1V8" V 6000 4150 50  0000 C CNN
 F 2 "" H 6000 3900 50  0001 C CNN
@@
 	5300 3550 5500 3550
 $Comp
-L power:GND #PWR023
+L power:GND #PWR022
 U 1 1 60AA905C
 P 6100 3550
-F 0 "#PWR023" H 6100 3300 50  0001 C CNN
+F 0 "#PWR022" H 6100 3300 50  0001 C CNN
 F 1 "GND" V 6100 3350 50  0000 C CNN
 F 2 "" H 6100 3550 50  0001 C CNN
@@
 Wire Wire Line
 	5500 3550 5700 3550
-$Comp
-L Logic_LevelTranslator:TXS0108EPW U1
-U 1 1 60AF84A4
-P 3250 3850
-F 0 "U1" H 3000 4500 50  0000 C CNN
-F 1 "TXS0108EPW" H 2900 3150 50  0000 C CNN
-F 2 "Package_SO:TSSOP-20_4.4x6.5mm_P0.65mm" H 3250 3100 50  0001 C CNN
-F 3 "www.ti.com/lit/ds/symlink/txs0108e.pdf" H 3250 3750 50  0001 C CNN
-	1    3250 3850
-	-1   0    0    -1
-$EndComp
 Wire Wire Line
 	5250 4150 5300 4150
@@
 Wire Wire Line
 	3250 4550 3250 4650
-Text GLabel 3850 3950 3    50   Input ~ 0
+Text GLabel 3850 4250 3    50   Input ~ 0
 FLASH_NSS
-Text GLabel 3950 3950 3    50   Input ~ 0
+Text GLabel 3950 4250 3    50   Input ~ 0
 FLASH_SCK
-Text GLabel 4150 3950 3    50   Input ~ 0
+Text GLabel 4150 4250 3    50   Input ~ 0
 FLASH_MOSI
-Text GLabel 4050 3950 3    50   Input ~ 0
+Text GLabel 4050 4250 3    50   Input ~ 0
 FLASH_MISO
 Text GLabel 5250 4550 0    50   Input ~ 0
@@
 Text GLabel 6150 4550 2    50   Input ~ 0
 FLASH_MISO
-NoConn ~ 2850 3950
-NoConn ~ 2850 4050
-NoConn ~ 2850 4150
-NoConn ~ 2850 4250
-NoConn ~ 3650 3950
-NoConn ~ 3650 4050
-NoConn ~ 3650 4150
-NoConn ~ 3650 4250
 Wire Wire Line
 	3650 3550 3850 3550
-Wire Wire Line
-	3650 3650 3950 3650
-Wire Wire Line
-	3650 3750 4050 3750
-Wire Wire Line
-	3650 3850 4150 3850
 $Comp
 L Device:R R10
@@
 $EndComp
 Wire Wire Line
-	3750 3250 3750 3450
-Wire Wire Line
-	3750 3450 3650 3450
-Wire Wire Line
 	3850 3250 3850 3550
-Connection ~ 3850 3550
-Wire Wire Line
-	3850 3550 3850 3950
-Wire Wire Line
-	3950 3250 3950 3650
-Connection ~ 3950 3650
-Wire Wire Line
-	3950 3650 3950 3950
-Wire Wire Line
-	4050 3250 4050 3750
-Connection ~ 4050 3750
-Wire Wire Line
-	4050 3750 4050 3950
-Wire Wire Line
-	4150 3250 4150 3850
-Connection ~ 4150 3850
-Wire Wire Line
-	4150 3850 4150 3950
 Wire Wire Line
 	3750 2950 3750 2850
@@
 	2750 3550 2850 3550
 Wire Wire Line
-	2850 3650 2750 3650
-Wire Wire Line
-	2750 3750 2850 3750
-Wire Wire Line
-	2850 3850 2750 3850
+	2850 3750 2750 3750
+Wire Wire Line
+	2750 3950 2850 3950
+Wire Wire Line
+	2850 4150 2750 4150
 $Comp
 L power:+3.3V #PWR03
@@
 $EndComp
 $Comp
-L power:GND #PWR020
+L power:GND #PWR019
 U 1 1 60CFA445
 P 5900 2850
-F 0 "#PWR020" H 5900 2600 50  0001 C CNN
+F 0 "#PWR019" H 5900 2600 50  0001 C CNN
 F 1 "GND" V 5905 2722 50  0000 R CNN
 F 2 "" H 5900 2850 50  0001 C CNN
@@
 $EndComp
 $Comp
-L power:GND #PWR019
+L power:GND #PWR018
 U 1 1 60D095DF
 P 5900 2450
-F 0 "#PWR019" H 5900 2200 50  0001 C CNN
+F 0 "#PWR018" H 5900 2200 50  0001 C CNN
 F 1 "GND" V 5905 2322 50  0000 R CNN
 F 2 "" H 5900 2450 50  0001 C CNN
@@
 	0    -1   -1   0
 $EndComp
+$Comp
+L Logic_LevelTranslator:TXB0104PW U1
+U 1 1 60AC3318
+P 3250 3850
+F 0 "U1" H 3450 3150 50  0000 C CNN
+F 1 "TXB0104PW" H 3000 3150 50  0000 C CNN
+F 2 "Package_SO:TSSOP-14_4.4x5mm_P0.65mm" H 3250 3100 50  0001 C CNN
+F 3 "http://www.ti.com/lit/ds/symlink/txb0104.pdf" H 3360 3945 50  0001 C CNN
+	1    3250 3850
+	-1   0    0    -1
+$EndComp
+Wire Wire Line
+	3850 3550 3850 4250
+Connection ~ 3850 3550
+Wire Wire Line
+	3750 3250 3750 3350
+Wire Wire Line
+	3750 3350 3650 3350
+Wire Wire Line
+	3950 3250 3950 3750
+Wire Wire Line
+	3650 3750 3950 3750
+Connection ~ 3950 3750
+Wire Wire Line
+	3950 3750 3950 4250
+Wire Wire Line
+	3650 3950 4050 3950
+Wire Wire Line
+	4050 3250 4050 3950
+Connection ~ 4050 3950
+Wire Wire Line
+	4050 3950 4050 4250
+Wire Wire Line
+	3650 4150 4150 4150
+Wire Wire Line
+	4150 3250 4150 4150
+Connection ~ 4150 4150
+Wire Wire Line
+	4150 4150 4150 4250
 $EndSCHEMATC
